File: pcb/daughter-board/daughter-board.kicad_sch (KiCad schematic)
At the start: 11 parts, among them J1 Conn_01x06_MountingPin, J2 USB_C_Receptacle_USB2.0_16P, J4 4P4C_Shielded, U1 SRV05-4

Commit message: schematics review with scgh
Parts:
- removed D1: D_Schottky, Diode_SMD:D_SOD-123, symbol Device:D_Schottky
- added C1: 100n, Capacitor_SMD:C_0603_1608Metric, symbol Device:C_Small
- added R3: 220k, Resistor_SMD:R_0603_1608Metric, symbol Device:R_Small
Connections:
- net VBUS is gone; now on net +5V: J2.A4 (VBUS), J2.A9 (VBUS), J2.B4 (VBUS), J2.B9 (VBUS)
- net GND: now also C1.2, R3.1; no longer J2.S1 (SHIELD)
- new net: C1.1, J2.S1 (SHIELD), R3.2
Other:
- note added: "CHECK mode and value"
- moved on the sheet: H1, H2, H3, H4

Commit message: layout ready for review
Parts:
- removed H1, H2, H3, H4: MountingHole, MountingHole:MountingHole_2.2mm_M2, symbol Mechanical:MountingHole
- removed J4: 4P4C_Shielded, Connector_RJ:RJ9_Evercom_5301-440xxx_Horizontal, symbol Connector:4P4C
- added C2, C3, C4, C5: 100n, Capacitor_SMD:C_0603_1608Metric, symbol Device:C_Small
- added H1, H2, H3, H4: MountingHole_Pad, MountingHole:MountingHole_2.2mm_M2_DIN965_Pad_TopBottom, symbol Mechanical:MountingHole_Pad
- added J3: PJ-320A, lib-zegonix:TRRS_Receptable, symbol lib_zegonix:TRRS_Receptacle
- added R4, R5, R6, R7: 330, Resistor_SMD:R_0603_1608Metric, symbol Device:R_Small
- R3: value 220k -> 330
Connections:
- net +5V: now also J3.T
- net GND: now also R3.2, C2.2, C3.2, C4.2, C5.2, J3.S, R4.2, R5.2, R6.2, R7.2; no longer R3.1
- net SPLIT_RX: now also J3.R2
- net SPLIT_TX: now also J3.R1
- net at C1.1, J2.S1 (SHIELD): now also R3.1; no longer R3.2
- new net: C4.1, H3.1, R6.1
- new net: C3.1, H2.1, R5.1
- new net: C2.1, H1.1, R4.1
- new net: C5.1, H4.1, R7.1
Other:
- note removed: "CHECK mode and value"
- moved on the sheet: R3
