File: pcb/pcb-qua-ken/pcb-quaken.kicad_pcb (KiCad board)
At the start: 2 copper layers, 142.4 x 115.9 mm, 91 parts, among them J1 Conn_01x06_MountingPin, J2 Conn_01x02_Pin, J3 Conn_01x04_Pin, SW1 SW_Push, SW2 Rotary_Encoder_Default, U1 XC6206PxxxMR, U2 STM32F401RCTx, Y1 12MHz

Commit message: schematics review with scgh
Other:
- board text added: "supply through pads of bypass caps"
Changed lines of the file:
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@@
   (gr_circle (center 151.592513 98.737488) (end 161.592513 98.737488)
     (stroke (width 0.15) (type default)) (fill none) (layer "User.1"))
+  (gr_text "supply through pads of bypass caps\n" (at 129.54 73.66) (layer "F.Fab")
+    (effects (font (size 1 1) (thickness 0.15)) (justify left bottom))
+  )
   (via (at 145.115 77.115) (size 0.8) (drill 0.4) (layers "F.Cu" "B.Cu") (net 1))
   (via (at 138.565 74.09) (size 0.8) (drill 0.4) (layers "F.Cu" "B.Cu") (net 1))
@@
   (segment (start 150.1025 58.945001) (end 150.0825 58.965001) (width 0.3) (layer "F.Cu") (net 4))
   (via (at 151.04 61.44) (size 0.8) (drill 0.4) (layers "F.Cu" "B.Cu") (net 4))
-  (segment (start 139.89 79.69) (end 139.89 77.129339) (width 0.3) (layer "B.Cu") (net 4))
   (segment (start 148.06188 77.04) (end 152.19 77.04) (width 0.3) (layer "B.Cu") (net 4))
+  (segment (start 143.065 80.755) (end 140.955 80.755) (width 0.3) (layer "B.Cu") (net 4))
   (segment (start 151.04 61.44) (end 152.59 61.44) (width 0.3) (layer "B.Cu") (net 4))
-  (segment (start 143.065 80.755) (end 140.955 80.755) (width 0.3) (layer "B.Cu") (net 4))
   (segment (start 139.984339 75.045) (end 139.89 75.045) (width 0.3) (layer "B.Cu") (net 4))
   (segment (start 154.34 66.29) (end 153.015 67.615) (width 0.3) (layer "B.Cu") (net 4))
   (segment (start 154.34 63.19) (end 154.34 66.29) (width 0.3) (layer "B.Cu") (net 4))
-  (segment (start 139.89 77.129339) (end 140.979339 76.04) (width 0.3) (layer "B.Cu") (net 4))
   (segment (start 152.59 61.44) (end 154.34 63.19) (width 0.3) (layer "B.Cu") (net 4))
+  (segment (start 140.955 80.755) (end 139.7 79.5) (width 0.3) (layer "B.Cu") (net 4))
   (segment (start 147.06188 76.04) (end 148.06188 77.04) (width 0.3) (layer "B.Cu") (net 4))
-  (segment (start 140.955 80.755) (end 139.89 79.69) (width 0.3) (layer "B.Cu") (net 4))
   (segment (start 152.19 77.04) (end 153.015 77.865) (width 0.3) (layer "B.Cu") (net 4))
+  (segment (start 139.7 79.5) (end 139.7 77.319339) (width 0.3) (layer "B.Cu") (net 4))
   (segment (start 140.979339 76.04) (end 139.984339 75.045) (width 0.3) (layer "B.Cu") (net 4))
   (segment (start 153.015 77.865) (end 153.015 78.965) (width 0.3) (layer "B.Cu") (net 4))
   (segment (start 153.84 77.04) (end 153.015 77.865) (width 0.3) (layer "B.Cu") (net 4))
+  (segment (start 139.7 77.319339) (end 140.979339 76.04) (width 0.3) (layer "B.Cu") (net 4))
   (segment (start 147.015 78.965) (end 147.015 78.08688) (width 0.3) (layer "B.Cu") (net 4))
   (segment (start 147.015 78.08688) (end 148.06188 77.04) (width 0.3) (layer "B.Cu") (net 4))

Commit message: layout ready for review
Parts:
- removed the C2 at (121.6, 71.3)
- added R1: 1k, Resistor_SMD:R_0402_1005Metric, B.Cu at (58.2, 82.7)
- added R3: 1k, Resistor_SMD:R_0402_1005Metric, B.Cu at (56.2, 80.1)
- added R4: 1k, Resistor_SMD:R_0402_1005Metric, B.Cu at (56.2, 78.8)
- C1, C10, C8, C9, MX19, SW1, U1: moved to B.Cu
- C11: value 4.7 -> 100n
- R2: value 5.1k -> 1k; moved to B.Cu
- moved R2 105.4 mm to (58.2, 81.4)
- moved J3 99.0 mm to (72.4, 42.2), turned to -90 degrees
- moved C10 89.2 mm to (73.4, 57.3)
- moved C8 86.9 mm to (64.6, 49.7), turned to -90 degrees
- moved MX29 86.3 mm to (63.0, 132.8)
- moved D29 86.1 mm to (70.1, 130.4)
- moved R8 85.8 mm to (58.9, 92.1)
- moved R9 85.8 mm to (58.9, 94.5)
- moved SW2 85.8 mm to (58.9, 97.3)
- moved D1 85.5 mm to (191.2, 48.2)
- moved D10 85.5 mm to (134.1, 60.1)
- moved D11 85.5 mm to (115.0, 62.4)
- moved D13 85.5 mm to (191.2, 86.3)
- moved D14 85.5 mm to (172.2, 86.3)
- moved D15 85.5 mm to (153.1, 81.5)
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- renumbered C3 to C2, C4 to C3, C5 to C4, C6 to C5, C7 to C6, C14 to C7, J2 to J1, J1 to J2, R9 to R10, R10 to R11, R5 to R12, R11 to R13, R3 to R5, R4 to R6, R6 to R7, R7 to R8, R8 to R9
Connections:
- D1 pad 1: unconnected-(D1-K-Pad1) -> /ROW0
- D10 pad 1: unconnected-(D10-K-Pad1) -> /ROW1
- D11 pad 1: unconnected-(D11-K-Pad1) -> /ROW1
- D12 pad 1: unconnected-(D12-K-Pad1) -> /ROW1
- D13 pad 1: unconnected-(D13-K-Pad1) -> /ROW2
- D14 pad 1: unconnected-(D14-K-Pad1) -> /ROW2
- D15 pad 1: unconnected-(D15-K-Pad1) -> /ROW2
- D16 pad 1: unconnected-(D16-K-Pad1) -> /ROW2
- D17 pad 1: unconnected-(D17-K-Pad1) -> /ROW2
- D18 pad 1: unconnected-(D18-K-Pad1) -> /ROW2
- D19 pad 1: unconnected-(D19-K-Pad1) -> /ROW3
- D2 pad 1: unconnected-(D2-K-Pad1) -> /ROW0
- D20 pad 1: unconnected-(D20-K-Pad1) -> /ROW3
- D21 pad 1: unconnected-(D21-K-Pad1) -> /ROW3
- D22 pad 1: unconnected-(D22-K-Pad1) -> /ROW3
- D23 pad 1: unconnected-(D23-K-Pad1) -> /ROW3
- D24 pad 1: unconnected-(D24-K-Pad1) -> /ROW3
- D25 pad 1: unconnected-(D25-K-Pad1) -> /ROW4
- D26 pad 1: unconnected-(D26-K-Pad1) -> /ROW4
- D27 pad 1: unconnected-(D27-K-Pad1) -> /ROW4
- D28 pad 1: unconnected-(D28-K-Pad1) -> /ROW4
- D29 pad 1: unconnected-(D29-K-Pad1) -> /ROW4
- D3 pad 1: unconnected-(D3-K-Pad1) -> /ROW0
- D30 pad 1: unconnected-(D30-K-Pad1) -> /ROW4
- D4 pad 1: unconnected-(D4-K-Pad1) -> /ROW0
- D5 pad 1: unconnected-(D5-K-Pad1) -> /ROW0
- D6 pad 1: unconnected-(D6-K-Pad1) -> /ROW0
- D7 pad 1: unconnected-(D7-K-Pad1) -> /ROW1
- D8 pad 1: unconnected-(D8-K-Pad1) -> /ROW1
- D9 pad 1: unconnected-(D9-K-Pad1) -> /ROW1
- MX1 pad 1: unconnected-(MX1-Pad1) -> /COL0
- MX10 pad 1: unconnected-(MX10-Pad1) -> /COL3
- MX11 pad 1: unconnected-(MX11-Pad1) -> /COL4
- MX12 pad 1: unconnected-(MX12-Pad1) -> /COL5
- MX13 pad 1: unconnected-(MX13-Pad1) -> /COL0
- MX14 pad 1: unconnected-(MX14-Pad1) -> /COL1
- MX15 pad 1: unconnected-(MX15-Pad1) -> /COL2
- MX16 pad 1: unconnected-(MX16-Pad1) -> /COL3
- MX17 pad 1: unconnected-(MX17-Pad1) -> /COL4
- MX18 pad 1: unconnected-(MX18-Pad1) -> /COL5
- MX19 pad 1: unconnected-(MX19-Pad1) -> /COL0
- MX2 pad 1: unconnected-(MX2-Pad1) -> /COL1
- MX20 pad 1: unconnected-(MX20-Pad1) -> /COL1
- MX21 pad 1: unconnected-(MX21-Pad1) -> /COL2
- MX22 pad 1: unconnected-(MX22-Pad1) -> /COL3
- MX23 pad 1: unconnected-(MX23-Pad1) -> /COL4
- MX24 pad 1: unconnected-(MX24-Pad1) -> /COL5
- MX25 pad 1: unconnected-(MX25-Pad1) -> /COL0
- MX26 pad 1: unconnected-(MX26-Pad1) -> /COL1
- MX27 pad 1: unconnected-(MX27-Pad1) -> /COL2
- MX28 pad 1: unconnected-(MX28-Pad1) -> /COL3
- MX29 pad 1: unconnected-(MX29-Pad1) -> /COL4
- MX3 pad 1: unconnected-(MX3-Pad1) -> /COL2
- MX4 pad 1: unconnected-(MX4-Pad1) -> /COL3
- MX5 pad 1: unconnected-(MX5-Pad1) -> /COL4
- MX6 pad 1: unconnected-(MX6-Pad1) -> /COL5
- MX7 pad 1: unconnected-(MX7-Pad1) -> /COL0
- MX8 pad 1: unconnected-(MX8-Pad1) -> /COL1
- MX9 pad 1: unconnected-(MX9-Pad1) -> /COL2
- R2 pad 1: +5V -> /SPLIT_RX
- R2 pad 2: /nRESET -> Net-(U2-PA2)
- SW2 pad S1: /ENC_SW_1 -> /ENC_SW_2
- SW2 pad S2: /ENC_SW_2 -> /COL5
- U2 pad 16: /SPLIT_TX -> Net-(U2-PA2)
- U2 pad 17: /SPLIT_RX -> Net-(U2-PA3)
- U2 pad 29: /COL2 -> unconnected-(U2-PB10-Pad29)
- U2 pad 33: /COL3 -> unconnected-(U2-PB12-Pad33)
- U2 pad 34: /COL4 -> unconnected-(U2-PB13-Pad34)
- U2 pad 35: /COL5 -> unconnected-(U2-PB14-Pad35)
- U2 pad 50: unconnected-(U2-PA15-Pad50) -> /COL2
- U2 pad 51: unconnected-(U2-PC10-Pad51) -> /COL3
- U2 pad 52: unconnected-(U2-PC11-Pad52) -> /COL4
- U2 pad 53: unconnected-(U2-PC12-Pad53) -> /COL5
- U2 pad 8: /ENC_A -> /ENC_B
- U2 pad 9: /ENC_B -> /ENC_A
Routing:
- net /COL0: track 0.00 -> 221.4 mm, vias 0 -> 8
- net /COL1: track 0.00 -> 200.0 mm, vias 0 -> 8
- net /COL2: track 0.00 -> 176.1 mm, vias 0 -> 9
- net /ROW4: track 0.00 -> 174.7 mm, vias 0 -> 3
- net /COL3: track 0.00 -> 167.5 mm, vias 0 -> 9
- net /COL4: track 0.00 -> 158.9 mm, vias 0 -> 9
- net /ROW0: track 0.00 -> 152.1 mm, vias 0 -> 2
- net /ROW3: track 0.00 -> 146.2 mm, vias 0 -> 2
- net /ROW1: track 0.00 -> 132.8 mm, vias 0 -> 2
- net /ROW2: track 0.00 -> 130.5 mm
- net /COL5: track 0.00 -> 77.9 mm, vias 0 -> 7
- net +3V3: track 43.2 -> 104.3 mm, vias 1 -> 3
- net /nRESET: track 0.00 -> 36.9 mm, vias 0 -> 2
- net /SWDIO: track 0.00 -> 33.3 mm, vias 0 -> 1
- net /SWCLK: track 0.00 -> 28.7 mm, vias 0 -> 1
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- added copper zone on B.Cu, net GND
Other:
- board size 142.4 x 115.9 mm -> 143.4 x 118.9 mm
- board text removed: "supply through pads of bypass caps"

Commit message: removed one switch from the thumb cluster
Parts:
- removed D25: D_Small, Diode_SMD:D_SOD-123
- removed MX25: MX_SW_HS, PCM_marbastlib-mx:SW_MX_HS_1u
Routing:
- net /COL0: track 221.4 -> 171.8 mm, vias 8 -> 6
- net /ROW4: track 174.7 -> 154.6 mm
- net Net-(D25-A): track 5.45 -> 0.00 mm
Other:
- outline, holes or cut-outs redrawn
