File: plate/plate.kicad_pcb (KiCad board)
At the start: 2 copper layers, 231.1 x 152.7 mm, 28 parts

Commit message: finalised first version of pcbs for prototype order added openscad file for the left halfs case
Parts:
- added MX29: Cutout, lib-zegonix:MX-SW-1u-Plate-Cutout, F.Cu at (194.6, 138.7)
- moved MX7 144.2 mm to (73.4, 76.9)
- moved MX19 144.0 mm to (73.4, 115.0)
- moved MX13 132.7 mm to (73.4, 96.0)
- moved MX14 131.1 mm to (92.5, 96.0)
- moved MX21 129.9 mm to (111.5, 110.3)
- moved MX20 128.2 mm to (92.5, 115.0)
- moved MX25 121.4 mm to (111.5, 129.3)
- moved MX22 111.0 mm to (130.6, 107.9)
- moved MX26 107.5 mm to (130.6, 126.9)
- moved MX6 107.4 mm to (168.7, 55.5)
- moved MX15 101.2 mm to (111.5, 91.2)
- moved MX8 94.0 mm to (92.5, 76.9)
- moved MX27 92.7 mm to (149.6, 129.3)
- moved MX24 89.1 mm to (168.7, 112.7)
- moved MX5 87.5 mm to (149.6, 53.1)
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Other:
- board size 231.1 x 152.7 mm -> 149.4 x 110.3 mm
