File: plate/plate.kicad_sch (KiCad schematic)
At the start: 28 parts

Commit message: finalised first version of pcbs for prototype order added openscad file for the left halfs case
Parts:
- added MX25: Cutout, lib-zegonix:MX-SW-1u-Plate-Cutout, symbol lib-zegonix:MX-SW-1u-Plate-Cutout
- renumbered MX25 to MX26, MX26 to MX27, MX27 to MX28, MX28 to MX29
Changed lines of the file:
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@@
 		(dnp no)
 		(fields_autoplaced yes)
-		(property "Reference" "MX28"
+		(property "Reference" "MX29"
 			(at 149.86 87.6299 0)
 			(effects
@@
 			(project "plate-left"
 				(path "/f5d34910-a58b-4db3-a32f-fb609945106e"
-					(reference "MX28")
+					(reference "MX29")
 					(unit 1)
 				)
@@
 		(dnp no)
 		(fields_autoplaced yes)
-		(property "Reference" "MX26"
+		(property "Reference" "MX27"
 			(at 116.84 87.6299 0)
 			(effects
@@
 			(project "plate-left"
 				(path "/f5d34910-a58b-4db3-a32f-fb609945106e"
-					(reference "MX26")
+					(reference "MX27")
 					(unit 1)
 				)
@@
 		(dnp no)
 		(fields_autoplaced yes)
-		(property "Reference" "MX27"
+		(property "Reference" "MX28"
 			(at 133.35 87.6299 0)
 			(effects
@@
 			(project "plate-left"
 				(path "/f5d34910-a58b-4db3-a32f-fb609945106e"
-					(reference "MX27")
+					(reference "MX28")
 					(unit 1)
 				)
@@
 	(symbol
 		(lib_id "lib-zegonix:MX-SW-1u-Plate-Cutout")
+		(at 80.01 88.9 0)
+		(unit 1)
+		(exclude_from_sim no)
+		(in_bom yes)
+		(on_board yes)
+		(dnp no)
+		(fields_autoplaced yes)
+		(property "Reference" "MX25"
+			(at 83.82 87.6299 0)
+			(effects
+				(font
+					(size 1.27 1.27)
+				)
+				(justify left)
+			)
+		)
+		(property "Value" "Cutout"
+			(at 83.82 90.1699 0)
+			(effects
+				(font
+					(size 1.27 1.27)
+				)
+				(justify left)
+			)
+		)
+		(property "Footprint" "lib-zegonix:MX-SW-1u-Plate-Cutout"
+			(at 80.01 95.25 0)
+			(effects
+				(font
+					(size 1.27 1.27)
+				)
+				(hide yes)
+			)
+		)
+		(property "Datasheet" ""
+			(at 80.01 88.9 0)
+			(effects
+				(font
+					(size 1.27 1.27)
+				)
+				(hide yes)
+			)
+		)
+		(property "Description" ""
+			(at 80.01 88.9 0)
+			(effects
+				(font
+					(size 1.27 1.27)
+				)
+				(hide yes)
+			)
+		)
+		(instances
+			(project "plate-left"
+				(path "/f5d34910-a58b-4db3-a32f-fb609945106e"
+					(reference "MX25")
+					(unit 1)
+				)
+			)
+		)
+	)
+	(symbol
+		(lib_id "lib-zegonix:MX-SW-1u-Plate-Cutout")
 		(at 96.52 68.58 0)
 		(unit 1)
@@
 		(dnp no)
 		(fields_autoplaced yes)
-		(property "Reference" "MX25"
+		(property "Reference" "MX26"
 			(at 100.33 87.6299 0)
 			(effects
@@
 			(project "plate-left"
 				(path "/f5d34910-a58b-4db3-a32f-fb609945106e"
-					(reference "MX25")
-					(unit 1)
-				)
+					(reference "MX26")
+					(unit 1)
+				)
