File: pcb-left/pcb-left.kicad_sch (KiCad schematic)
At the start: 91 parts, among them J1 Conn_01x02_Pin, J2 Conn_01x06_MountingPin, J3 Conn_01x04_Pin, SW1 SW_Push, SW2 Rotary_Encoder_Default, U1 XC6206PxxxMR, U2 STM32F401RCTx, Y1 12MHz

Commit message: added new/renamed folders and files forgotten during last commits finished pcb-left
Connections:
- net COL0: now also U2.58 (PB6); no longer U2.61 (PB8)
- net COL1: now also U2.57 (PB5); no longer U2.62 (PB9)
- net COL2: now also U2.56 (PB4); no longer U2.50 (PA15)
- net COL3: now also U2.55 (PB3); no longer U2.51 (PC10)
- net COL4: now also U2.54 (PD2); no longer U2.52 (PC11)
Changed lines of the file:
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@@
   (no_connect (at 93.98 156.21))
   (no_connect (at 127 161.29))
-  (no_connect (at 127 143.51))
-  (no_connect (at 93.98 113.03))
   (no_connect (at 93.98 138.43))
   (no_connect (at 127 138.43))
@@
   (no_connect (at 127 90.17))
   (no_connect (at 127 135.89))
+  (no_connect (at 127 153.67))
   (no_connect (at 127 163.83))
   (no_connect (at 127 97.79))
-  (no_connect (at 127 148.59))
+  (no_connect (at 127 156.21))
   (no_connect (at 127 113.03))
   (no_connect (at 127 166.37))
+  (no_connect (at 93.98 143.51))
+  (no_connect (at 93.98 146.05))
   (no_connect (at 127 95.25))
   (no_connect (at 93.98 151.13))
   (no_connect (at 93.98 125.73))
-  (no_connect (at 127 140.97))
-  (no_connect (at 127 146.05))
+  (no_connect (at 127 128.27))
   (wire (pts (xy 87.63 170.815) (xy 87.63 161.29))
     (stroke (width 0) (type default))
@@
     (stroke (width 0) (type default))
   )
-  (wire (pts (xy 127 128.27) (xy 151.13 128.27))
-    (stroke (width 0) (type default))
-  )
   (wire (pts (xy 246.38 167.005) (xy 271.78 167.005))
     (stroke (width 0) (type default))
@@
     (stroke (width 0) (type default))
   )
-  (wire (pts (xy 66.675 143.51) (xy 93.98 143.51))
-    (stroke (width 0) (type default))
-  )
   (wire (pts (xy 156.21 212.09) (xy 156.21 216.535))
     (stroke (width 0) (type default))
@@
     (stroke (width 0) (type default))
   )
-  (wire (pts (xy 127 156.21) (xy 151.13 156.21))
-    (stroke (width 0) (type default))
-  )
   (wire (pts (xy 120.65 50.8) (xy 120.65 56.515))
     (stroke (width 0) (type default))
@@
     (stroke (width 0) (type default))
   )
+  (wire (pts (xy 127 140.97) (xy 151.13 140.97))
+    (stroke (width 0) (type default))
+  )
   (wire (pts (xy 246.38 108.585) (xy 303.53 108.585))
     (stroke (width 0) (type default))
@@
     (stroke (width 0) (type default))
   )
-  (wire (pts (xy 66.675 146.05) (xy 93.98 146.05))
-    (stroke (width 0) (type default))
-  )
   (wire (pts (xy 66.675 95.25) (xy 93.98 95.25))
     (stroke (width 0) (type default))
@@
     (stroke (width 0) (type default))
   )
+  (wire (pts (xy 66.675 113.03) (xy 93.98 113.03))
+    (stroke (width 0) (type default))
+  )
   (wire (pts (xy 109.22 83.82) (xy 106.68 83.82))
     (stroke (width 0) (type default))
@@
     (stroke (width 0) (type default))
   )
+  (wire (pts (xy 127 148.59) (xy 151.13 148.59))
+    (stroke (width 0) (type default))
+  )
   (wire (pts (xy 120.65 34.29) (xy 120.65 40.64))
     (stroke (width 0) (type default))
@@
     (stroke (width 0) (type default))
   )
+  (wire (pts (xy 127 143.51) (xy 151.13 143.51))
+    (stroke (width 0) (type default))
+  )
   (wire (pts (xy 262.255 242.57) (xy 262.255 245.11))
     (stroke (width 0) (type default))
@@
     (stroke (width 0) (type default))
   )
+  (wire (pts (xy 127 146.05) (xy 151.13 146.05))
+    (stroke (width 0) (type default))
+  )
   (wire (pts (xy 328.93 139.7) (xy 328.93 156.845))
     (stroke (width 0) (type default))
@@
   )
   (wire (pts (xy 278.13 139.7) (xy 278.13 156.845))
-    (stroke (width 0) (type default))
-  )
-  (wire (pts (xy 127 153.67) (xy 151.13 153.67))
     (stroke (width 0) (type default))
   )
@@
     (effects (font (size 1.27 1.27)) (justify left bottom))
   )
-  (label "COL4" (at 66.675 146.05 0) (fields_autoplaced)
+  (label "COL4" (at 66.675 113.03 0) (fields_autoplaced)
     (effects (font (size 1.27 1.27)) (justify left bottom))
   )
@@
     (effects (font (size 1.27 1.27)) (justify left bottom))
   )
-  (label "COL1" (at 151.13 156.21 180) (fields_autoplaced)
+  (label "COL1" (at 151.13 146.05 180) (fields_autoplaced)
     (effects (font (size 1.27 1.27)) (justify right bottom))
   )
@@
     (effects (font (size 1.27 1.27)) (justify left bottom))
   )
-  (label "COL0" (at 151.13 153.67 180) (fields_autoplaced)
+  (label "COL0" (at 151.13 148.59 180) (fields_autoplaced)
     (effects (font (size 1.27 1.27)) (justify right bottom))
   )
@@
     (effects (font (size 1.27 1.27)) (justify left bottom))
   )
-  (label "COL3" (at 66.675 143.51 0) (fields_autoplaced)
-    (effects (font (size 1.27 1.27)) (justify left bottom))
-  )
-  (label "COL2" (at 151.13 128.27 180) (fields_autoplaced)
-    (effects (font (size 1.27 1.27)) (justify right bottom))
-  )
+  (label "COL3" (at 151.13 140.97 180) (fields_autoplaced)
+    (effects (font (size 1.27 1.27)) (justify right bottom))
+  )
+  (label "COL2" (at 151.13 143.51 180) (fields_autoplaced)
+    (effects (font (size 1.27 1.27)) (justify right bottom))
+  )

Commit message: quick save
Parts:
- removed R10, R8: 5.1k, Resistor_SMD:R_0603_1608Metric, symbol Device:R_Small
- removed R12: 1k, Resistor_SMD:R_0603_1608Metric, symbol Device:R_Small
- added C14: 100n, Capacitor_SMD:C_0603_1608Metric, symbol Device:C_Small
- added D30: ~, lib-zegonix:SK6812MINI-E_3.2x2.8_reverse_mount, symbol lib-zegonix:sk6812mini-e
- C12, C13: value 22p -> 12p
- J2: footprint Connector_JST:JST_SHL_SM06B-SHLS-TF_1x06-1MP_P1.00mm_Horizontal -> Connector_JST:JST_SH_SM06B-SRSS-TB_1x06-1MP_P1.00mm_Horizontal
- R1, R2: value 27 -> 10k
- R11, R13, R7, R9: value 5.1k -> 10k
- SW2: now not fitted; now left out of the parts list
- Y1: value 12MHz -> 8MHz
Connections:
- net +3V3: now also J1.1 (Pin_1), C14.1, D30.1 (VDD)
- net ENC_A: now also R9.2
- net ENC_B: now also R11.1
- net GND: now also R1.2, R2.2, C14.2, D30.3 (GND); no longer J1.2 (Pin_2)
- net USB_D+: now also U2.45 (PA12); no longer R2.1
- net USB_D-: now also U2.44 (PA11); no longer R1.1
- net XOUT: now also C13.2, Y1.1
- net BOOT1: now reaches U2.28 (PB2)
- net BOOT1: now also R2.1
- net IND_LED: now reaches U2.34 (PB13)
- net IND_LED: now also D30.4 (DIN)
- net BOOTSEL renamed BOOT0
- net BOOT0: now also J1.2 (Pin_2), R1.1; no longer J1.1 (Pin_1)
- no-connect marks 26 -> 27
Other:
- note added: "Decoupling Capacitors for Pins 1, 13, 19, 32, 48, 64 + Bulk Capacitor"
- note removed: "C_l = 12pF"
- note removed: "Decoupling Capacitors for Pins 1, 19, 32, 48, 64 + Bulk Capacitor"
- note removed: "PB2 has alternate Function BOOT1"
- moved on the sheet: C1, C10, C11, C12, C13, C2, C3, C4, C5, C6, C7, C8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

Commit message: finalised first version of pcbs for prototype order added openscad file for the left halfs case
Parts:
- added D25: D_Small, Diode_SMD:D_SOD-123, symbol Device:D_Small
- added MX25: MX_SW_HS, PCM_marbastlib-mx:SW_MX_HS_1u, symbol PCM_marbastlib-mx:MX_SW_HS
- renumbered C9 to C10, C14 to C13, C13 to C14, C10 to C8, C8 to C9, D25 to D26, D26 to D27, D27 to D28, D28 to D29, D29 to D30, D30 to D31, J3 to J2, J2 to J3, MX25 to MX26, MX26 to MX27, MX27 to MX28, MX28 to MX29, R13 to R10, R9 to R8, R11 to R9
Connections:
- net COL0: now also U2.59 (PB7), MX25.1; no longer U2.58 (PB6)
- net COL1: now also U2.58 (PB6); no longer U2.57 (PB5)
- net COL2: now also U2.57 (PB5); no longer U2.56 (PB4)
- net ENC_A: now also U2.35 (PB14); no longer U2.9 (PC1)
- net ENC_B: now also U2.36 (PB15); no longer U2.8 (PC0)
- net HANDEDNESS: now also U2.11 (PC3); no longer U2.10 (PC2)
- net IND_LED: now also U2.10 (PC2); no longer U2.34 (PB13)
- net ROW0: now also U2.61 (PB8); no longer U2.26 (PB0)
- net ROW1: now also U2.56 (PB4); no longer U2.25 (PC5)
- net ROW2: now also U2.52 (PC11); no longer U2.24 (PC4)
- net ROW3: now also U2.51 (PC10); no longer U2.23 (PA7)
- net ROW4: now also U2.50 (PA15), D25.1 (K); no longer U2.22 (PA6)
- new net: D25.2 (A), MX25.2

Commit message: intermediate save
Parts:
- added R11: 1k, Resistor_SMD:R_0603_1608Metric, symbol Device:R_Small
- MX1, MX10, MX11, MX12, MX13, MX14, MX15, MX16, MX17, MX18, MX19, MX2, MX20, MX21, MX22, MX23, MX24, MX25, MX26, MX27, MX28, MX29, MX3, MX4, MX5, MX6, MX7, MX8, MX9: footprint PCM_marbastlib-mx:SW_MX_HS_1u -> PCM_marbastlib-mx:SW_MX_HS_CPG151101S11_1u
- R4, R6: footprint Resistor_SMD:R_0402_1005Metric -> Resistor_SMD:R_0603_1608Metric; now in the parts list
Connections:
- net COL0: now also U2.17 (PA3); no longer U2.59 (PB7)
- net COL1: now also U2.20 (PA4); no longer U2.58 (PB6)
- net COL2: now also U2.21 (PA5); no longer U2.57 (PB5)
- net COL3: now also U2.22 (PA6); no longer U2.55 (PB3)
- net COL4: now also U2.23 (PA7); no longer U2.54 (PD2)
- net COL5: now also U2.41 (PA8); no longer U2.53 (PC12)
- net GND: now also R11.2; no longer SW1.1
- net HANDEDNESS: now also U2.16 (PA2); no longer U2.11 (PC3)
- net IND_LED: now also U2.15 (PA1); no longer U2.10 (PC2)
- net ROW0: now also U2.55 (PB3); no longer U2.61 (PB8)
- net ROW2: now also U2.57 (PB5); no longer U2.52 (PC11)
- net ROW3: now also U2.58 (PB6); no longer U2.51 (PC10)
- net ROW4: now also U2.59 (PB7); no longer U2.50 (PA15)
- new net: R11.1, SW1.1
Other:
- moved on the sheet: C11, C8, SW1, U2
